File: kicad/strata.kicad_pcb (KiCad board)
At the start: 2 copper layers, 302 x 110 mm, 376 parts, among them J1 Eurorack Mono Jack, J10 Conn_01x02_Male, J11 Conn_01x04_Male, J12 Conn_01x04_Female, J13 Conn_01x08_Male, J14 Eurorack Mono Jack, J15 Conn_01x08_Female, J16 Eurorack Mono Jack, J17 Eurorack Mono Jack, J18 Eurorack Mono Jack, J19 Eurorack Mono Jack, J2 Eurorack Mono Jack, J20 Eurorack Mono Jack, J21 Eurorack Mono Jack, J22 Eurorack Mono Jack, J23 Eurorack Mono Jack, J24 Eurorack Mono Jack, J25 Eurorack Mono Jack, J26 Eurorack Mono Jack, J27 Eurorack Mono Jack, J28 Eurorack Mono Jack, J29 Eurorack Mono Jack, J3 Eurorack Mono Jack, J30 Eurorack Mono Jack, J31 Eurorack Mono Jack, J32 Conn_01x08_Female, J33 Eurorack Mono Jack, J34 Conn_01x08_Male, J35 Conn_01x08_Female, J36 Conn_01x08_Male, J37 Eurorack Power Small, J38 Conn_02x04_Odd_Even, J4 Eurorack Mono Jack, J41 Conn_01x03_Male, J42 Conn_01x06_Female, J43 Eurorack Mono Jack, J44 Eurorack Mono Jack, J45 Eurorack Mono Jack, J46 Eurorack Mono Jack, J47 Eurorack Mono Jack, J48 Eurorack Mono Jack, J49 Eurorack Mono Jack, J5 Conn_01x04_Female, J50 Eurorack Mono Jack, J51 Eurorack Mono Jack, J52 Conn_01x04_Female, J53 Conn_01x04_Male, J6 Conn_01x06_Female, J7 Conn_01x04_Male, J8 Conn_01x06_Male, J9 Conn_01x02_Female, Q1 2N3904, Q10 2N3904, Q11 2N3906, Q12 2N3904, Q13 2N3906, Q14 2N3906, Q15 2N3904, Q16 2N3904, Q2 2N3904, Q3 2N3904, Q4 2N3904, Q5 2N3904, Q6 2N3904, Q7 2N3904, Q8 2N3904, Q9 2N3904, U1 TL072, U10 LM13700, U11 TL074, U12 CD4024, U13 TL072, U14 4017, U15 4017, U16 4017, U17 4017, U18 TL074, U19 TL072, U2 L78L05_TO92, U20 TL074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

Commit message: component positioning mostly done
Parts:
- C1, C10, C11, C12, C16, C17, C19, C2, C29, C3, C30, C32, C33, C34, C35, C36, C37, C38, C39, C4, C41, C42, C43, C44, C46, C47, C48, C49, C50, C51, C55, C56, C57, C58, C59, C60, C61, C62, C63, C64, C65, C66, C67, C68, C8: footprint rumblesan-standard-parts:C_Rect_L7.0mm_W3.5mm_P5.00mm -> rumblesan-standard-parts:C_Rect_L7.0mm_W2.5mm_P5.00mm
- moved J42 605.1 mm to (302.7, 175.9)
- moved J43 605.1 mm to (321.6, 181.3)
- moved J44 605.1 mm to (332.6, 181.3)
- moved J45 605.1 mm to (305.9, 198.6)
- moved J46 605.1 mm to (317.0, 197.2)
- moved J47 605.1 mm to (310.5, 181.3)
- moved RV23 605.1 mm to (329.4, 195.1)
- moved R141 44.6 mm to (211.1, 107.2), turned to 0 degrees
- moved J11 42.5 mm to (211.8, 110.5), turned to 90 degrees
- moved J12 42.4 mm to (59.8, 110.5), turned to -90 degrees
- moved R120 34.7 mm to (81.3, 66.3), turned to 90 degrees
- moved R137 34.2 mm to (211.1, 98.0), turned to 0 degrees
- moved R142 32.3 mm to (221.2, 104.1), turned to 180 degrees
- moved R24 27.6 mm to (218.4, 120.1), turned to -90 degrees
- moved R47 25.4 mm to (266.2, 67.3), turned to 180 degrees
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Connections:
- J26 pad T: Net-(J32-Pad3) -> Net-(J26-PadT)
- J32 pad 3: Net-(J32-Pad3) -> Net-(J29-PadTN)
- J32 pad 4: Net-(J29-PadTN) -> unconnected-(J32-Pad4)
- J32 pad 5: Net-(J29-PadT) -> Net-(J32-Pad5)
- J32 pad 8: Net-(J32-Pad8) -> Net-(J26-PadT)
- J34 pad 3: /Filter VCA/VCA_INPUT -> /Filter VCA/AUDIO_INPUT1
- J34 pad 4: /Filter VCA/AUDIO_INPUT1 -> unconnected-(J34-Pad4)
- J34 pad 5: /Filter VCA/VCA_OUTPUT -> /VCA CV/VCA_CV_ATTV_TOP
- J34 pad 6: /VCA CV/VCA_LEVEL -> /VCA CV/VCA_CV_ATTV_BOTTOM
- J34 pad 7: /VCA CV/VCA_CV_ATTV_TOP -> /VCA CV/VCA_LEVEL
- J34 pad 8: /VCA CV/VCA_CV_ATTV_BOTTOM -> /Filter VCA/VCA_INPUT
- J35 pad 1: Net-(J35-Pad1) -> Net-(J29-PadT)
- J35 pad 2: Net-(RV19-Pad1) -> Net-(J35-Pad2)
- J35 pad 3: unconnected-(J35-Pad3) -> Net-(J35-Pad3)
- J36 pad 1: /Filter CV/RES_CV_ATTV_TOP -> /Filter VCA/VCA_OUTPUT
- J36 pad 2: /Filter CV/RES_CV_ATTV_BOTTOM -> /Filter CV/RES_CV_ATTV_TOP
- J36 pad 3: unconnected-(J36-Pad3) -> /Filter CV/RES_CV_ATTV_BOTTOM
- J6 pad 2: Net-(J6-Pad2) -> Net-(RV4-Pad3)
- J6 pad 3: Net-(J6-Pad3) -> Net-(RV4-Pad2)
- J6 pad 5: Net-(J6-Pad5) -> Net-(RV5-Pad2)
- J6 pad 6: Net-(J6-Pad6) -> Net-(RV6-Pad3)
- J8 pad 1: /Delay/FEEDBACK_SOURCE -> /Delay/DELAY_WET_MIX
- J8 pad 2: /Delay/FEEDBACK_MIX -> /Delay/FEEDBACK_SOURCE
- J8 pad 3: /Delay/DRY_AUDIO_SOURCE -> /Delay/FEEDBACK_MIX
- J8 pad 4: /Delay/DRY_AUDIO_MIX -> /Delay/DRY_AUDIO_SOURCE
- J8 pad 5: /Delay/DELAY_WET_SOURCE -> /Delay/DRY_AUDIO_MIX
- J8 pad 6: /Delay/DELAY_WET_MIX -> /Delay/DELAY_WET_SOURCE
- RV15 pad 2: Net-(J32-Pad6) -> Net-(J32-Pad7)
- RV16 pad 1: Net-(J32-Pad8) -> Net-(J32-Pad6)
- RV16 pad 3: Net-(J32-Pad7) -> Net-(J32-Pad5)
- RV19 pad 1: Net-(RV19-Pad1) -> Net-(J35-Pad3)
- RV19 pad 3: Net-(J35-Pad1) -> Net-(J35-Pad2)
- RV4 pad 2: Net-(J6-Pad2) -> Net-(RV4-Pad2)
- RV4 pad 3: Net-(J6-Pad1) -> Net-(RV4-Pad3)
- RV5 pad 2: Net-(J6-Pad4) -> Net-(RV5-Pad2)
- RV5 pad 3: Net-(J6-Pad3) -> Net-(J6-Pad4)
- RV6 pad 2: Net-(J6-Pad6) -> Net-(J6-Pad1)
- RV6 pad 3: Net-(J6-Pad5) -> Net-(RV6-Pad3)
