File: kicad/sub-dividers.kicad_sch (KiCad schematic)
At the start: 62 parts, among them Q2 2N3904, Q3 2N3904, Q4 2N3904, Q5 2N3904, Q6 2N3904, Q7 2N3904, Q8 2N3904, U13 TL072, U14 4017, U15 4017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

Commit message: component positioning mostly done
Parts:
- C49, C50: footprint rumblesan-standard-parts:C_Rect_L7.0mm_W3.5mm_P5.00mm -> rumblesan-standard-parts:C_Rect_L7.0mm_W2.5mm_P5.00mm
Changed lines of the file:
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@@
     (property "Reference" "C50" (id 0) (at 49.53 62.7212 90))
     (property "Value" "100nF" (id 1) (at 49.53 65.2581 90))
-    (property "Footprint" "rumblesan-standard-parts:C_Rect_L7.0mm_W3.5mm_P5.00mm" (id 2) (at 48.26 62.865 90)
-      (effects (font (size 1.27 1.27)) hide)
-    )
+    (property "Footprint" "rumblesan-standard-parts:C_Rect_L7.0mm_W2.5mm_P5.00mm" (id 2) (at 48.26 62.865 90))
     (property "Datasheet" "~" (id 3) (at 49.53 60.96 90)
       (effects (font (size 1.27 1.27)) hide)
@@
       (effects (font (size 1.27 1.27)) (justify left))
     )
-    (property "Footprint" "rumblesan-standard-parts:C_Rect_L7.0mm_W3.5mm_P5.00mm" (id 2) (at 46.355 204.47 90)
-      (effects (font (size 1.27 1.27)) hide)
-    )
+    (property "Footprint" "rumblesan-standard-parts:C_Rect_L7.0mm_W2.5mm_P5.00mm" (id 2) (at 46.355 204.47 90)
+      (effects (font (size 1.27 1.27)) hide)
+    )

Commit message: initial layout done
Parts:
- added C5, C69, C70, C71: 100nF, rumblesan-standard-parts:C_Rect_L7.0mm_W2.5mm_P5.00mm, symbol rumblesan-standard-parts:C
Connections:
- net GND: now also C5.1, C69.1, C70.1, C71.1
- net VCC: now also C5.2, C69.2, C70.2, C71.2

Commit message: Full rejig to use attiny for divider
Parts:
- C49, C5, C50, C69, C70, C71: Spec ceramic C0G -> ceramic X7R
Changed lines of the file:
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@@
       (effects (font (size 1.27 1.27)) hide)
     )
-    (property "Spec" "ceramic C0G" (id 4) (at 49.53 64.77 90)
+    (property "Spec" "ceramic X7R" (id 4) (at 49.53 64.77 90)
       (effects (font (size 1.27 1.27)) hide)
     )
@@
       (effects (font (size 1.27 1.27)) hide)
     )
-    (property "Spec" "ceramic C0G" (id 4) (at 152.4 105.41 90)
+    (property "Spec" "ceramic X7R" (id 4) (at 152.4 105.41 90)
       (effects (font (size 1.27 1.27)) hide)
     )
@@
       (effects (font (size 1.27 1.27)) hide)
     )
-    (property "Spec" "ceramic C0G" (id 4) (at 44.45 205.74 90)
+    (property "Spec" "ceramic X7R" (id 4) (at 44.45 205.74 90)
       (effects (font (size 1.27 1.27)) hide)
     )
@@
       (effects (font (size 1.27 1.27)) hide)
     )
-    (property "Spec" "ceramic C0G" (id 4) (at 232.41 105.41 90)
+    (property "Spec" "ceramic X7R" (id 4) (at 232.41 105.41 90)
       (effects (font (size 1.27 1.27)) hide)
     )
@@
       (effects (font (size 1.27 1.27)) hide)
     )
-    (property "Spec" "ceramic C0G" (id 4) (at 97.79 105.41 90)
+    (property "Spec" "ceramic X7R" (id 4) (at 97.79 105.41 90)
       (effects (font (size 1.27 1.27)) hide)
     )
@@
       (effects (font (size 1.27 1.27)) hide)
     )
-    (property "Spec" "ceramic C0G" (id 4) (at 289.56 105.41 90)
-      (effects (font (size 1.27 1.27)) hide)
-    )
+    (property "Spec" "ceramic X7R" (id 4) (at 289.56 105.41 90)
+      (effects (font (size 1.27 1.27)) hide)
+    )
