File: kicad/mercurial.kicad_sch (KiCad schematic)
At the start: 121 parts, among them J1 Eurorack Mono Jack, J10 Conn_01x04_Male, J11 Conn_01x04_Male, J12 Conn_01x04_Female, J13 Conn_01x08_Male, J14 Eurorack Mono Jack, J15 Conn_01x08_Female, J16 Eurorack Mono Jack, J17 Eurorack Mono Jack, J18 Eurorack Mono Jack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

Commit message: geographically reannotate parts
Parts:
- renumbered C1 to C3, C3 to C5, C73 to C6, C7 to C62, C6 to C63, D2 to D20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
