File: kicad/divider.kicad_sch (KiCad schematic)
At the start: 9 parts, among them J39 SPI, Q6 2N3904, Q8 2N3904, U11 ATtiny24A-P, U14 74LS241

Commit message: Changes after investigations and tweaking
Parts:
- removed J39: SPI, Connector_PinHeader_2.54mm:PinHeader_2x03_P2.54mm_Vertical, symbol Connector_Generic:Conn_02x03_Odd_Even
- added J39: AVR-ISP-6, Connector_PinHeader_2.54mm:PinHeader_2x03_P2.54mm_Vertical, symbol Connector:AVR-ISP-6
- added R131: 100k, Rumblesan_Standard_Parts:R_Axial_DIN0207_L6.3mm_D2.5mm_P10.16mm_Horizontal, symbol Rumblesan Standard Parts:R
Connections:
- net +5V: now also J39.2 (VCC), R131.2
- net GND: now also J39.6 (GND)
- net IC_DIV_OUT_5: now also J39.4 (MOSI)
- net IC_DIV_OUT_7: now also J39.1 (MISO)
- net RST renamed IC_RESET
- net IC_RESET: now also J39.5 (~{RST}), R131.1
- net SCK renamed IC_SCK
- net IC_SCK: now also J39.3 (SCK)
- no-connect marks 2 -> 1
