File: kicad/filter-cv.kicad_sch (KiCad schematic)
At the start: 21 parts, among them Q10 2N3904, Q11 2N3906, Q9 2N3906, U16 TL074

Commit message: Changes after investigations and tweaking
Parts:
- added D13: 1N4148, Rumblesan_Standard_Parts:D_DO-35_SOD27_P7.62mm_Horizontal, symbol Device:D
- added R132: 1k, Rumblesan_Standard_Parts:R_Axial_DIN0207_L6.3mm_D2.5mm_P10.16mm_Horizontal, symbol Rumblesan Standard Parts:R
- R114: value 20k -> 33k
- R122: value 100k -> 330k
- R123: value 180k -> 220k
- R125, R126: value 20k -> 100k
Connections:
- net GND: now also R132.1
- net RES_CV_ATTV_TOP: now also D13.1 (K)
- net at Q11.1 (E), R114.1: now also R132.2
- net at C58.2, Q11.2 (B), U16.1: now also D13.2 (A)
Other:
- note added: "aim for i_res range of 0.0 to 0.4ma with higher resonance at lower i_res"
- note added: "i_res ma = Vc/330k * (R1k + 33k)/1k"
- moved on the sheet: R114
