File: kicad/noise.kicad_sch (KiCad schematic)
At the start: 9 parts, among them Q1 BC547, Q2 BC549C

Commit message: Changes after investigations and tweaking
Parts:
- RV1: value 200kB -> 200k
Changed lines of the file:
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@@
       (effects (font (size 1.27 1.27)) (justify right))
     )
-    (property "Value" "200kB" (at 85.09 69.215 0)
+    (property "Value" "200k" (at 85.09 69.215 0)
       (effects (font (size 1.27 1.27)) (justify right))
     )
