File: kicad/ouroboros.kicad_sch (KiCad schematic)
At the start: 121 parts, among them J1 Eurorack Mono Jack, J10 Conn_01x03_Male, J11 Eurorack Mono Jack, J12 Eurorack Mono Jack, J13 Eurorack Mono Jack, J14 Eurorack Mono Jack, J19 Eurorack Mono Jack, J2 Eurorack Mono Jack, J20 Eurorack Mono Jack, J21 Eurorack Mono Jack, J22 Eurorack Mono Jack, J23 Eurorack Mono Jack, J24 Eurorack Mono Jack, J25 Eurorack Mono Jack, J26 Eurorack Mono Jack, J27 Eurorack Mono Jack, J28 Conn_01x06_Male, J29 Conn_01x04_Male, J3 Eurorack Mono Jack, J30 Conn_01x04_Male, J31 Conn_01x04_Male, J32 Conn_01x06_Male, J33 Conn_01x04_Male, J34 Conn_01x08_Male, J35 Conn_01x08_Male, J36 Eurorack Power Small, J38 Conn_02x04_Odd_Even, J4 Eurorack Mono Jack, J40 Conn_01x08_Female, J41 Conn_01x08_Female, J42 Conn_01x04_Female, J43 Conn_01x06_Female, J44 Conn_01x04_Female, J45 Conn_01x04_Female, J46 Conn_01x04_Female, J47 Conn_01x06_Female, J5 Eurorack Mono Jack, J6 Eurorack Mono Jack, J7 Eurorack Mono Jack, J8 Eurorack Mono Jack, J9 Eurorack Mono Jack, U1 TL074, U8 L78L05_TO92

Commit message: Changes after investigations and tweaking
Parts:
- R34: value 100k -> 330k
Other:
- moved on the sheet: RV20
Changed lines of the file:
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@@
     (stroke (width 0) (type default))
   )
-  (wire (pts (xy 327.66 64.77) (xy 327.66 95.25))
+  (wire (pts (xy 327.66 68.58) (xy 327.66 95.25))
     (stroke (width 0) (type default))
   )
@@
     (stroke (width 0) (type default))
   )
-  (wire (pts (xy 307.34 68.58) (xy 307.34 71.12))
+  (wire (pts (xy 318.77 72.39) (xy 318.77 73.66))
     (stroke (width 0) (type default))
   )
@@
     (stroke (width 0) (type default))
   )
+  (wire (pts (xy 318.77 63.5) (xy 318.77 64.77))
+    (stroke (width 0) (type default))
+  )
   (wire (pts (xy 172.72 167.64) (xy 172.72 172.72))
     (stroke (width 0) (type default))
@@
     (stroke (width 0) (type default))
   )
-  (wire (pts (xy 307.34 58.42) (xy 307.34 60.96))
-    (stroke (width 0) (type default))
-  )
   (wire (pts (xy 120.65 31.75) (xy 124.46 31.75))
     (stroke (width 0) (type default))
@@
     (stroke (width 0) (type default))
   )
-  (wire (pts (xy 311.15 64.77) (xy 327.66 64.77))
+  (wire (pts (xy 322.58 68.58) (xy 327.66 68.58))
     (stroke (width 0) (type default))
   )
@@
     (effects (font (size 1.27 1.27)) (justify left bottom))
   )
+  (netclass_flag "" (length 2.54) (shape round) (at 368.3 57.15 0) (fields_autoplaced)
+    (effects (font (size 1.27 1.27)) (justify left bottom))
+    (property "Netclass" "Power" (at 368.9096 54.61 0)
+      (effects (font (size 1.27 1.27) italic) (justify left))
+    )
+  )
   (netclass_flag "" (length 2.54) (shape round) (at 372.11 29.21 0) (fields_autoplaced)
     (effects (font (size 1.27 1.27)) (justify left bottom))
@@
       (effects (font (size 1.27 1.27)) hide)
     )
-    (property "Name" "Stability Noise Level" (at 33.02 62.23 0)
+    (property "Name" "Stability Noise Level" (at 34.29 62.23 0)
       (effects (font (size 1.27 1.27)))
     )
@@
     )
   )
-  (symbol (lib_id "Rumblesan Standard Parts:R_Potentiometer") (at 307.34 64.77 0) (unit 1)
+  (symbol (lib_id "Rumblesan Standard Parts:R_Potentiometer") (at 318.77 68.58 0) (unit 1)
     (in_bom yes) (on_board yes) (dnp no)
-    (property "Reference" "RV20" (at 305.5621 65.6047 0)
+    (property "Reference" "RV20" (at 316.9921 69.4147 0)
       (effects (font (size 1.27 1.27)) (justify right))
     )
-    (property "Value" "100kB" (at 305.5621 63.0678 0)
+    (property "Value" "100kB" (at 316.9921 66.8778 0)
       (effects (font (size 1.27 1.27)) (justify right))
     )
-    (property "Footprint" "Rumblesan_Standard_Parts:Potentiometer_Alpha_RD901F-40-00D_Single_Vertical" (at 297.18 66.04 90)
+    (property "Footprint" "Rumblesan_Standard_Parts:Potentiometer_Alpha_RD901F-40-00D_Single_Vertical" (at 308.61 69.85 90)
       (effects (font (size 1.27 1.27)) hide)
     )
-    (property "Datasheet" "http://www.taiwanalpha.com/downloads?target=products&id=113" (at 299.72 64.77 90)
+    (property "Datasheet" "http://www.taiwanalpha.com/downloads?target=products&id=113" (at 311.15 68.58 90)
       (effects (font (size 1.27 1.27)) hide)
     )
-    (property "Name" "Filter Resonance" (at 316.23 59.69 0)
+    (property "Name" "Filter Resonance" (at 309.88 62.23 0)
       (effects (font (size 1.27 1.27)))
     )
@@
       (effects (font (size 1.27 1.27)) (justify right))
     )
-    (property "Value" "100k" (at 293.37 68.58 90)
+    (property "Value" "330k" (at 293.37 68.58 90)
       (effects (font (size 1.27 1.27)) (justify right))
     )
@@
     )
   )
-  (symbol (lib_id "power:VCC") (at 307.34 58.42 0) (unit 1)
+  (symbol (lib_id "power:VCC") (at 318.77 63.5 0) (unit 1)
     (in_bom yes) (on_board yes) (dnp no) (fields_autoplaced)
-    (property "Reference" "#PWR050" (at 307.34 62.23 0)
+    (property "Reference" "#PWR050" (at 318.77 67.31 0)
       (effects (font (size 1.27 1.27)) hide)
     )
-    (property "Value" "VCC" (at 307.34 54.8442 0)
+    (property "Value" "VCC" (at 318.77 59.9242 0)
       (effects (font (size 1.27 1.27)))
     )
-    (property "Footprint" "" (at 307.34 58.42 0)
+    (property "Footprint" "" (at 318.77 63.5 0)
       (effects (font (size 1.27 1.27)) hide)
     )
-    (property "Datasheet" "" (at 307.34 58.42 0)
+    (property "Datasheet" "" (at 318.77 63.5 0)
       (effects (font (size 1.27 1.27)) hide)
     )
@@
     )
   )
-  (symbol (lib_id "power:GND") (at 307.34 71.12 0) (unit 1)
+  (symbol (lib_id "power:GND") (at 318.77 73.66 0) (unit 1)
     (in_bom yes) (on_board yes) (dnp no) (fields_autoplaced)
-    (property "Reference" "#PWR051" (at 307.34 77.47 0)
+    (property "Reference" "#PWR051" (at 318.77 80.01 0)
       (effects (font (size 1.27 1.27)) hide)
     )
-    (property "Value" "GND" (at 307.34 75.5634 0)
+    (property "Value" "GND" (at 318.77 78.1034 0)
       (effects (font (size 1.27 1.27)))
     )
-    (property "Footprint" "" (at 307.34 71.12 0)
+    (property "Footprint" "" (at 318.77 73.66 0)
       (effects (font (size 1.27 1.27)) hide)
     )
-    (property "Datasheet" "" (at 307.34 71.12 0)
+    (property "Datasheet" "" (at 318.77 73.66 0)
       (effects (font (size 1.27 1.27)) hide)
     )
