File: kicad/ouroboros.kicad_sch (KiCad schematic)
At the start: 121 parts, among them J1 Eurorack Mono Jack, J10 Conn_01x03_Male, J11 Eurorack Mono Jack, J12 Eurorack Mono Jack, J13 Eurorack Mono Jack, J14 Eurorack Mono Jack, J19 Eurorack Mono Jack, J2 Eurorack Mono Jack, J20 Eurorack Mono Jack, J21 Eurorack Mono Jack, J22 Eurorack Mono Jack, J23 Eurorack Mono Jack, J24 Eurorack Mono Jack, J25 Eurorack Mono Jack, J26 Eurorack Mono Jack, J27 Eurorack Mono Jack, J28 Conn_01x06_Male, J29 Conn_01x04_Male, J3 Eurorack Mono Jack, J30 Conn_01x04_Male, J31 Conn_01x04_Male, J32 Conn_01x06_Male, J33 Conn_01x04_Male, J34 Conn_01x08_Male, J35 Conn_01x08_Male, J36 Eurorack Power Small, J38 Conn_02x04_Odd_Even, J4 Eurorack Mono Jack, J40 Conn_01x08_Female, J41 Conn_01x08_Female, J42 Conn_01x04_Female, J43 Conn_01x06_Female, J44 Conn_01x04_Female, J45 Conn_01x04_Female, J46 Conn_01x04_Female, J47 Conn_01x06_Female, J5 Eurorack Mono Jack, J6 Eurorack Mono Jack, J7 Eurorack Mono Jack, J8 Eurorack Mono Jack, J9 Eurorack Mono Jack, U1 TL074, U8 L78L05_TO92

Commit message: Removing test points from BOM
Parts:
- TP1, TP10, TP11, TP13, TP14, TP16, TP2, TP3, TP4, TP5, TP6, TP7, TP9: now left out of the parts list
Changed lines of the file:
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@@
   )
   (symbol (lib_id "Connector:TestPoint") (at 372.11 16.51 270) (unit 1)
-    (in_bom yes) (on_board yes) (dnp no) (fields_autoplaced)
+    (in_bom no) (on_board yes) (dnp no) (fields_autoplaced)
     (property "Reference" "TP4" (at 376.809 15.6753 90)
       (effects (font (size 1.27 1.27)) (justify left))
@@
   )
   (symbol (lib_id "Connector:TestPoint") (at 120.65 20.32 0) (unit 1)
-    (in_bom yes) (on_board yes) (dnp no) (fields_autoplaced)
+    (in_bom no) (on_board yes) (dnp no) (fields_autoplaced)
     (property "Reference" "TP9" (at 122.047 16.1833 0)
       (effects (font (size 1.27 1.27)) (justify left))
@@
   )
   (symbol (lib_id "Connector:TestPoint") (at 325.12 237.49 0) (unit 1)
-    (in_bom yes) (on_board yes) (dnp no)
+    (in_bom no) (on_board yes) (dnp no)
     (property "Reference" "TP14" (at 323.85 232.41 0)
       (effects (font (size 1.27 1.27)) (justify left))
@@
   )
   (symbol (lib_id "Connector:TestPoint") (at 369.57 50.8 270) (unit 1)
-    (in_bom yes) (on_board yes) (dnp no) (fields_autoplaced)
+    (in_bom no) (on_board yes) (dnp no) (fields_autoplaced)
     (property "Reference" "TP11" (at 374.269 49.9653 90)
       (effects (font (size 1.27 1.27)) (justify left))
@@
   )
   (symbol (lib_id "Connector:TestPoint") (at 368.3 116.84 90) (unit 1)
-    (in_bom yes) (on_board yes) (dnp no) (fields_autoplaced)
+    (in_bom no) (on_board yes) (dnp no) (fields_autoplaced)
     (property "Reference" "TP6" (at 364.998 112.5052 90)
       (effects (font (size 1.27 1.27)))
@@
   )
   (symbol (lib_id "Connector:TestPoint") (at 116.84 48.26 90) (unit 1)
-    (in_bom yes) (on_board yes) (dnp no) (fields_autoplaced)
+    (in_bom no) (on_board yes) (dnp no) (fields_autoplaced)
     (property "Reference" "TP10" (at 113.538 43.9252 90)
       (effects (font (size 1.27 1.27)))
@@
   )
   (symbol (lib_id "Connector:TestPoint") (at 382.27 25.4 270) (unit 1)
-    (in_bom yes) (on_board yes) (dnp no) (fields_autoplaced)
+    (in_bom no) (on_board yes) (dnp no) (fields_autoplaced)
     (property "Reference" "TP13" (at 386.969 24.5653 90)
       (effects (font (size 1.27 1.27)) (justify left))
@@
   )
   (symbol (lib_id "Connector:TestPoint") (at 375.92 34.29 270) (unit 1)
-    (in_bom yes) (on_board yes) (dnp no) (fields_autoplaced)
+    (in_bom no) (on_board yes) (dnp no) (fields_autoplaced)
     (property "Reference" "TP1" (at 380.619 33.4553 90)
       (effects (font (size 1.27 1.27)) (justify left))
@@
   )
   (symbol (lib_id "Connector:TestPoint") (at 364.49 177.8 270) (unit 1)
-    (in_bom yes) (on_board yes) (dnp no) (fields_autoplaced)
+    (in_bom no) (on_board yes) (dnp no) (fields_autoplaced)
     (property "Reference" "TP7" (at 369.189 176.9653 90)
       (effects (font (size 1.27 1.27)) (justify left))
@@
   )
   (symbol (lib_id "Connector:TestPoint") (at 368.3 124.46 90) (unit 1)
-    (in_bom yes) (on_board yes) (dnp no) (fields_autoplaced)
+    (in_bom no) (on_board yes) (dnp no) (fields_autoplaced)
     (property "Reference" "TP5" (at 364.998 120.1252 90)
       (effects (font (size 1.27 1.27)))
@@
   )
   (symbol (lib_id "Connector:TestPoint") (at 318.77 237.49 0) (unit 1)
-    (in_bom yes) (on_board yes) (dnp no)
+    (in_bom no) (on_board yes) (dnp no)
     (property "Reference" "TP2" (at 317.5 232.41 0)
       (effects (font (size 1.27 1.27)) (justify left))
@@
   )
   (symbol (lib_id "Connector:TestPoint") (at 93.98 62.23 270) (unit 1)
-    (in_bom yes) (on_board yes) (dnp no) (fields_autoplaced)
+    (in_bom no) (on_board yes) (dnp no) (fields_autoplaced)
     (property "Reference" "TP16" (at 98.679 61.3953 90)
       (effects (font (size 1.27 1.27)) (justify left))
@@
   )
   (symbol (lib_id "Connector:TestPoint") (at 331.47 237.49 0) (unit 1)
-    (in_bom yes) (on_board yes) (dnp no)
+    (in_bom no) (on_board yes) (dnp no)
     (property "Reference" "TP3" (at 330.2 232.41 0)
       (effects (font (size 1.27 1.27)) (justify left))

Commit message: Changing decoupling caps to ceramic X7R
Parts:
- C4, C5: Spec ceramic C0G -> ceramic X7R
Changed lines of the file:
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@@
       (effects (font (size 1.27 1.27)) hide)
     )
-    (property "Spec" "ceramic C0G" (at 100.33 139.7 90)
+    (property "Spec" "ceramic X7R" (at 100.33 139.7 90)
       (effects (font (size 1.27 1.27)) hide)
     )
@@
       (effects (font (size 1.27 1.27)) hide)
     )
-    (property "Spec" "ceramic C0G" (at 100.33 127 90)
-      (effects (font (size 1.27 1.27)) hide)
-    )
+    (property "Spec" "ceramic X7R" (at 100.33 127 90)
+      (effects (font (size 1.27 1.27)) hide)
+    )

Commit message: Updating board for new footprint libraries
Parts:
- C3, C4, C5, C6: symbol Rumblesan Standard Parts:C -> Rumblesan_Standard_Parts:C
- C62, C63: footprint Rumblesan_Standard_Parts:CP_Radial_D5.0mm_L11.0mm_P2.00mm_Horizontal -> Rumblesan_Standard_Parts:CP_Radial_D5.0mm_P2.00mm; symbol Rumblesan Standard Parts:C_Polarized -> Rumblesan_Standard_Parts:C_Polarized
- J1, J11, J12, J13, J14, J19, J2, J20, J21, J22, J23, J24, J25, J26, J27, J3, J4, J5, J6, J7, J8, J9: footprint Rumblesan_Standard_Parts:Jack_3.5mm_QingPu_WQP-PJ398SM_Vertical -> Rumblesan_Audio_Connectors:Jack_3.5mm_QingPu_WQP-PJ398SM_Vertical; symbol Audio_Connectors:Eurorack_Mono_Jack -> Connector_Audio:AudioJack2_SwitchT
- J36: footprint Eurorack_Power:Eurorack_PowerHeader_2x05_P2.54mm_Shrouded -> Rumblesan_Eurorack_Power:Eurorack_PowerHeader_2x05_P2.54mm_Shrouded; symbol Eurorack_Power:Eurorack Power Small -> Rumblesan_Eurorack_Power:Eurorack Power Small
- R1, R10, R11, R13, R14, R15, R16, R17, R18, R19, R2, R20, R21, R22, R23, R24, R25, R26, R27, R32, R34, R35, R39, R40, R41, R42, R43, R44, R45, R46, R5, R7, R8, R9, R99: symbol Rumblesan Standard Parts:R -> Rumblesan_Standard_Parts:R
- RV10, RV11, RV12, RV13, RV14, RV18, RV19, RV2, RV20, RV21, RV3, RV4, RV5, RV6, RV7: footprint Rumblesan_Standard_Parts:Potentiometer_Alpha_RD901F-40-00D_Single_Vertical -> Rumblesan_Potentiometer_THT:Potentiometer_Alpha_RD901F-40-00D_Single_Vertical; symbol Rumblesan Standard Parts:R_Potentiometer -> Rumblesan_Standard_Parts:R_Potentiometer
- RV8: footprint Rumblesan_Standard_Parts:Potentiometer_Alpha_RD901F-40-00D_Single_Vertical -> Rumblesan_Potentiometer_THT:Potentiometer_Alpha_RD901F-40-00D_Single_Vertical; symbol Rumblesan Standard Parts:R_Potentiometer -> Rumblesan_Standard_Parts:R_Potentiometer; Name (none) -> Delay Time CV Attenuverter
- RV9: footprint Rumblesan_Standard_Parts:Potentiometer_Alpha_RD901F-40-00D_Single_Vertical -> Rumblesan_Potentiometer_THT:Potentiometer_Alpha_RD901F-40-00D_Single_Vertical; symbol Rumblesan Standard Parts:R_Potentiometer -> Rumblesan_Standard_Parts:R_Potentiometer; Name (none) -> Delay Time
- U1: footprint Rumblesan_Standard_Parts:DIP-14_W7.62mm_Socket -> Package_DIP:DIP-14_W7.62mm_Socket
- U8: footprint Rumblesan_Standard_Parts:TO-92_Inline_Wide -> Package_TO_SOT_THT:TO-92_Inline_Wide
Connections:
- net CV Mixer/CV_MIX_IN_1: now also J9.TN; no longer J9.3 (Tip_normalize)
- net CV Mixer/CV_MIX_OUT: now also J14.TN; no longer J14.3 (Tip_normalize)
- net GND: now also J1.S, J11.S, J12.S, J13.S, J14.S, J19.S, J2.S, J20.S, J21.S, J22.S, J23.S, J24.S, J25.S, J26.S, J27.S, J3.S, J4.S, J5.S, J6.S, J7.S, J8.S, J9.S; no longer J1.1 (Sleeve), J11.1 (Sleeve), J12.1 (Sleeve), J13.1 (Sleeve), J14.1 (Sleeve), J19.1 (Sleeve), J2.1 (Sleeve), J20.1 (Sleeve), J21.1 (Sleeve), J22.1 (Sleeve), J23.1 (Sleeve), J24.1 (Sleeve), J25.1 (Sleeve), J26.1 (Sleeve), J27.1 (Sleeve), J3.1 (Sleeve), J4.1 (Sleeve), J5.1 (Sleeve), J6.1 (Sleeve), J7.1 (Sleeve), J8.1 (Sleeve), J9.1 (Sleeve)
- net at RV12.3: now also J12.T; no longer J12.2 (Tip)
- net at R41.1: now also J19.T; no longer J19.2 (Tip)
- net at J41.1 (Pin_1): now also J22.T; no longer J22.2 (Tip)
- net at R5.1: now also J1.T; no longer J1.2 (Tip)
- net at RV2.3: now also J2.T; no longer J2.2 (Tip)
- net at R32.1: now also J14.T; no longer J14.2 (Tip)
- net at J45.1 (Pin_1): now also J9.T; no longer J9.2 (Tip)
- net at R42.1: now also J25.T; no longer J25.2 (Tip)
- net at J41.3 (Pin_3), R42.2: now also J13.TN; no longer J13.3 (Tip_normalize)
- net at R35.1: now also J21.T; no longer J21.2 (Tip)
- net at R39.1: now also J20.T; no longer J20.2 (Tip)
- net at R19.1: now also J8.T; no longer J8.2 (Tip)
- net at R13.1: now also J7.TN; no longer J7.3 (Tip_normalize)
- net at R22.1: now also J4.T; no longer J4.2 (Tip)
- net at J46.2 (Pin_2), R2.1: now also J2.TN; no longer J2.3 (Tip_normalize)
- net at J46.4 (Pin_4), R8.2: now also J5.TN; no longer J5.3 (Tip_normalize)
- net at R2.2: now also J3.T; no longer J3.2 (Tip)
- net at J43.6 (Pin_6): now also J12.TN; no longer J12.3 (Tip_normalize)
- net at R8.1: now also J6.T; no longer J6.2 (Tip)
- net at R44.1: now also J23.T; no longer J23.2 (Tip)
- net at R34.1: now also J13.T; no longer J13.2 (Tip)
- net at R40.1, R45.2: now also J27.T; no longer J27.2 (Tip)
- net at RV5.3: now also J5.T; no longer J5.2 (Tip)
- net at J41.2 (Pin_2), R43.2: now also J27.TN; no longer J27.3 (Tip_normalize)
- net at J41.5 (Pin_5), R46.2: now also J8.TN; no longer J8.3 (Tip_normalize)
- net at J43.2 (Pin_2): now also J7.T; no longer J7.2 (Tip)
- net at J43.5 (Pin_5): now also J11.TN; no longer J11.3 (Tip_normalize)
- net at R43.1: now also J26.T; no longer J26.2 (Tip)
- net at R46.1: now also J24.T; no longer J24.2 (Tip)
- net at R27.1: now also J11.T; no longer J11.2 (Tip)
Other:
- moved on the sheet: J1, J19, J20, J21, J22, J23, J24, J25, J26, R1, R10, R11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
