File: kicad/delay.kicad_sch (KiCad schematic)
At the start: 61 parts, among them Q3 2N3904, U3 4020, U4 TL072, U5 TL074, U6 PT2399

Commit message: More layout tweaks
Parts:
- TP15: value DelayInputAudioTestPoint -> TestPoint
Changed lines of the file:
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@@
 		(on_board yes)
 		(dnp no)
-		(fields_autoplaced yes)
 		(property "Reference" "TP15"
 			(at 157.099 77.9053 90)
@@
 			)
 		)
-		(property "Value" "DelayInputAudioTestPoint"
+		(property "Value" "TestPoint"
 			(at 157.099 80.4422 90)
 			(effects
@@
 				)
 				(justify left)
+				(hide yes)
 			)
 		)
@@
 			)
 		)
-		(property "Description" ""
-			(at 152.4 78.74 0)
+		(property "Description" "Delay Input"
+			(at 155.194 75.438 90)
 			(effects
 				(font
 					(size 1.27 1.27)
 				)
-				(hide yes)
 			)
 		)
