File: kicad/filter-vca.kicad_sch (KiCad schematic)
At the start: 42 parts, among them U10 TL074, U15 TL072, U17 SSI2164

Commit message: More layout tweaks
Connections:
- net GND: now also C55.2; no longer C55.1
- net VEE: now also C55.1; no longer C55.2
Other:
- moved on the sheet: C55
Changed lines of the file:
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@@
 	(symbol
 		(lib_id "Rumblesan_Standard_Parts:C")
-		(at 297.18 43.18 0)
+		(at 297.18 43.18 180)
 		(unit 1)
 		(exclude_from_sim no)
@@
 					(size 1.27 1.27)
 				)
-				(justify left)
+				(justify right)
 			)
 		)
@@
 					(size 1.27 1.27)
 				)
-				(justify left)
+				(justify right)
 			)
 		)
 		(property "Footprint" "Rumblesan_Standard_Parts:C_Rect_L7.0mm_W2.5mm_P5.00mm"
-			(at 302.895 41.91 0)
+			(at 291.465 44.45 0)
 			(effects
 				(font
@@
 		)
 		(property "Datasheet" "~"
-			(at 304.8 43.18 0)
+			(at 289.56 43.18 0)
 			(effects
 				(font
@@
 		)
 		(property "Spec" "ceramic X7R"
-			(at 300.99 43.18 90)
+			(at 293.37 43.18 90)
 			(effects
 				(font
@@
 		)
 		(property "Tolerance" "5%"
-			(at 300.99 34.925 90)
+			(at 293.37 51.435 90)
 			(effects
 				(font
